File: cbEval.UIFaceI2C.Busses.kicad_sch (KiCad schematic)
At the start: 25 parts, among them J1 Bergstik-II_3, J2 Bergstik-II_3, J3 Header.Hor.2x8.9-103326-0-08, J4 Header.Hor.2x8.9-103326-0-08, J5 Socket.Hor.2x8.1-5535512-8, J6 Bergstik-II_3, J7 Bergstik-II_6, J8 Bergstik-II_3, J9 Socket.Hor.2x8.1-5535512-8

Commit message: Bauteile aktualisiert
Parts:
- C1: ID X7R-5.4n7 -> (none); MPN (none) -> X7R-5.4n7
- J1, J2, J6, J8: value Bergstik-II_3 -> Bergstik-II_1x3; ID 68000-103HLF -> (none); MPN (none) -> 68000-103HLF
- J3, J4: ID 9-103326-0-08 -> (none); MPN (none) -> 9-103326-0-08
- J5, J9: ID 1-5535512-8 -> (none); MPN (none) -> 1-5535512-8
- J7: value Bergstik-II_6 -> Bergstik-II_1x6; ID 68000-106HLF -> (none); MPN (none) -> 68000-106HLF
- JP1: ID 68000-102HLF -> (none); MPN (none) -> 68000-102HLF
- R1, R10, R12, R2, R3, R6, R9: value 10k -> 10K; ID MFR-25FBF52-10K -> (none); MPN (none) -> MFR-25FBF52-10K
- R11: value 4k7 -> 4K7; ID MFR-25FBF52-4K7 -> (none); MPN (none) -> MFR-25FBF52-4K7
- R4, R5: ID MFR-25FBF52-47K5 -> (none); MPN (none) -> MFR-25FBF52-47K5
- R7, R8: ID MFR-25FBF52-60R4 -> (none); MPN (none) -> MFR-25FBF52-60R4
- S1, S2: ID JS202011CQN -> (none); MPN (none) -> JS202011CQN
