File: cbEval.UIFaceI2C.Display.kicad_sch (KiCad schematic)
At the start: 15 parts, among them J11 Bergstik-II_1x3, U4 TN0702N3-G, U5 TN0702N3-G

Commit message: Bauteile aktualisiert
Parts:
- C2, C3, C4, C5, C6, C7, C8: ID TAP105K035SCS -> (none); MPN (none) -> TAP105K035SCS
- DS1: ID EA DOGM204W-A -> (none); MPN (none) -> EA DOGM204W-A
- J11: ID 68000-103HLF -> (none); MPN (none) -> 68000-103HLF
- R22: ID MFR-25FBF52-24R -> (none); MPN (none) -> MFR-25FBF52-24R
- R23: ID MFR-25FBF52-18R -> (none); MPN (none) -> MFR-25FBF52-18R
- R24, R25: ID MFR-25FBF52-47K5 -> (none); MPN (none) -> MFR-25FBF52-47K5
- U4, U5: ID TN0702N3-G -> (none); MPN (none) -> TN0702N3-G
Changed lines of the file:
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@@
 			)
 		)
-		(property "ID" "TAP105K035SCS"
+		(property "MPN" "TAP105K035SCS"
 			(at 146.05 93.98 90)
 			(effects
@@
 			)
 		)
-		(property "ID" "68000-103HLF"
+		(property "MPN" "68000-103HLF"
 			(at 57.15 71.12 90)
 			(effects
@@
 			)
 		)
-		(property "ID" "TAP105K035SCS"
+		(property "MPN" "TAP105K035SCS"
 			(at 100.33 93.98 90)
 			(effects
@@
 			)
 		)
-		(property "ID" "TAP105K035SCS"
+		(property "MPN" "TAP105K035SCS"
 			(at 163.83 93.98 90)
 			(effects
@@
 			)
 		)
-		(property "ID" "MFR-25FBF52-24R"
+		(property "MPN" "MFR-25FBF52-24R"
 			(at 215.9 76.2 90)
-			(do_not_autoplace yes)
 			(effects
 				(font
@@
 			)
 		)
-		(property "ID" "MFR-25FBF52-47K5"
-			(at 203.2 132.08 90)
-			(do_not_autoplace yes)
-			(effects
-				(font
-					(size 0.635 0.635)
-					(italic yes)
-				)
-			)
-		)
 		(property "Package" "D0207"
 			(at 208.28 132.08 0)
@@
 			)
 		)
+		(property "MPN" "MFR-25FBF52-47K5"
+			(at 203.2 132.08 90)
+			(effects
+				(font
+					(size 0.635 0.635)
+					(italic yes)
+				)
+			)
+		)
 		(pin "1"
 		)
@@
 			)
 		)
-		(property "ID" "MFR-25FBF52-18R"
-			(at 193.04 76.2 90)
-			(do_not_autoplace yes)
-			(effects
-				(font
-					(size 0.635 0.635)
-					(italic yes)
-				)
-			)
-		)
 		(property "Package" "D0207"
 			(at 198.12 76.2 0)
@@
 			)
 		)
+		(property "MPN" "MFR-25FBF52-18R"
+			(at 193.04 76.2 90)
+			(effects
+				(font
+					(size 0.635 0.635)
+					(italic yes)
+				)
+			)
+		)
 		(pin "2"
 		)
@@
 			)
 		)
-		(property "ID" "TAP105K035SCS"
+		(property "MPN" "TAP105K035SCS"
 			(at 69.85 93.98 90)
 			(effects
@@
 			)
 		)
-		(property "ID" "TAP105K035SCS"
+		(property "MPN" "TAP105K035SCS"
 			(at 130.81 93.98 90)
 			(effects
@@
 			)
 		)
-		(property "ID" "EA DOGM204W-A"
+		(property "MPN" "EA DOGM204W-A"
 			(at 119.38 43.18 0)
 			(effects
@@
 			)
 		)
-		(property "ID" "MFR-25FBF52-47K5"
-			(at 180.34 132.08 90)
-			(do_not_autoplace yes)
-			(effects
-				(font
-					(size 0.635 0.635)
-					(italic yes)
-				)
-			)
-		)
 		(property "Package" "D0207"
 			(at 185.42 132.08 0)
@@
 			)
 		)
+		(property "MPN" "MFR-25FBF52-47K5"
+			(at 180.34 132.08 90)
+			(effects
+				(font
+					(size 0.635 0.635)
+					(italic yes)
+				)
+			)
+		)
 		(pin "1"
 		)
@@
 			)
 		)
-		(property "ID" "TAP105K035SCS"
+		(property "MPN" "TAP105K035SCS"
 			(at 85.09 93.98 90)
 			(effects
@@
 			)
 		)
-		(property "ID" "TAP105K035SCS"
+		(property "MPN" "TAP105K035SCS"
 			(at 115.57 93.98 90)
 			(effects
@@
 			)
 		)
-		(property "ID" "TN0702N3-G"
-			(at 198.12 111.76 90)
-			(effects
-				(font
-					(size 0.635 0.635)
-				)
-			)
-		)
 		(property "Voltage" "20V"
 			(at 200.66 114.3 0)
@@
 			)
 		)
+		(property "MPN" "TN0702N3-G"
+			(at 198.12 111.76 90)
+			(effects
+				(font
+					(size 0.635 0.635)
+				)
+			)
+		)
 		(pin "1"
 		)
@@
 			)
 		)
-		(property "ID" "TN0702N3-G"
-			(at 220.98 121.92 90)
-			(effects
-				(font
-					(size 0.635 0.635)
-				)
-			)
-		)
 		(property "Voltage" "20V"
 			(at 223.52 124.46 0)
@@
 			)
 		)
+		(property "MPN" "TN0702N3-G"
+			(at 220.98 121.92 90)
+			(effects
+				(font
+					(size 0.635 0.635)
+				)
+			)
+		)
