File: cbEval.UIFaceI2C.kicad_sch (KiCad schematic)
At the start: 20 parts, among them J10 Bergstik-II_1x3, U1 MCP23017-E/SP, U2 MCP23017-E/SP, U3 ATtiny85-20PU

Commit message: Bauteile aktualisiert
Parts:
- added J12: DIN41612.B.2x32.Male.Horizontal.THT, BTech.Connector.DIN41612:DIN41612.B.2x32.Male.Horizontal.THT, symbol J.DIN41612:DIN41612.B.2x32.Male.Horizontal.THT
- C9: ID X7R-5.100n -> (none); MPN (none) -> X7R-5.100n
- D1, D2, D3, D4: ID MV5439A -> (none); MPN (none) -> MV5439A
- H1: value CIME.E.BE3500S.2x -> CIME.E.BE3500S.4x; ID CIME/E/BE3500S -> (none); MPN (none) -> CIME/E/BE3500S
- J10: ID 68000-103HLF -> (none); MPN (none) -> 68000-103HLF
- R13, R14, R15, R16, R17, R18, R19, R20: ID MFR-25FBF52-1K -> (none); MPN (none) -> MFR-25FBF52-1K
- R21: ID MFR-25FBF52-10K -> (none); MPN (none) -> MFR-25FBF52-10K
- U1, U2: ID MCP23017-E/SP -> (none); MPN (none) -> MCP23017-E/SP
- U3: ID ATtiny85-20PU -> (none); MPN (none) -> ATtiny85-20PU

Commit message: Zwischenstand
Parts:
- added J13: DIN41612.B.2x32.Female.Horizontal.THT, BTech.Connector.DIN41612:DIN41612.B.2x32.Female.Horizontal.THT, symbol J.DIN41612:DIN41612.B.2x32.Female.Horizontal.THT
Changed lines of the file:
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@@
+	)
+	(symbol
+		(lib_id "J.DIN41612:DIN41612.B.2x32.Female.Horizontal.THT")
+		(at -3.81 105.41 0)
+		(mirror y)
+		(unit 1)
+		(exclude_from_sim no)
+		(in_bom yes)
+		(on_board yes)
+		(dnp no)
+		(property "Reference" "J13"
+			(at -8.89 19.05 0)
+			(effects
+				(font
+					(size 1.778 1.778)
+				)
+			)
+		)
+		(property "Value" "DIN41612.B.2x32.Female.Horizontal.THT"
+			(at -16.51 142.24 90)
+			(do_not_autoplace yes)
+			(effects
+				(font
+					(size 1.778 1.778)
+				)
+			)
+		)
+		(property "Footprint" "BTech.Connector.DIN41612:DIN41612.B.2x32.Female.Horizontal.THT"
+			(at -21.59 105.41 90)
+			(effects
+				(font
+					(size 1.016 1.016)
+				)
+				(hide yes)
+			)
+		)
+		(property "Datasheet" "https://www.hirose.com/product/document?clcode=CL0583-0079-9-72&productname=PCN10C-20S-2.54DSA(72)&series=PCN10&documenttype=Catalog&lang=en&documentid=D49718_en"
+			(at -19.05 105.41 90)
+			(effects
+				(font
+					(size 1.27 1.27)
+				)
+				(hide yes)
+			)
+		)
+		(property "Description" ""
+			(at -21.59 105.41 90)
+			(effects
+				(font
+					(size 1.27 1.27)
+				)
+				(hide yes)
+			)
+		)
+		(property "Package" "DIN41612.B.2x32.Female.Horizontal.THT"
+			(at -16.51 59.69 90)
+			(do_not_autoplace yes)
+			(effects
+				(font
+					(size 1.778 1.778)
+				)
+			)
+		)
+		(property "MPN" "  PCN13-64S-2.54DS(71)"
+			(at -8.89 189.23 0)
+			(effects
+				(font
+					(size 0.635 0.635)
+					(italic yes)
+				)
+			)
+		)
+		(property "Usage" "Usage"
+			(at -8.89 191.77 0)
+			(effects
+				(font
+					(size 1.27 1.27)
+				)
+			)
+		)
+		(property "Manufacturer" "Hirose Electric Co Ltd"
+			(at -24.13 105.41 90)
+			(effects
+				(font
+					(size 1.27 1.27)
+				)
+				(hide yes)
+			)
+		)
+		(pin "a9"
+		)
+		(pin "b12"
+		)
+		(pin "a26"
+		)
+		(pin "b4"
+		)
+		(pin "b9"
+		)
+		(pin "b17"
+		)
+		(pin "a27"
+		)
+		(pin "a29"
+		)
+		(pin "a25"
+		)
+		(pin "a28"
+		)
+		(pin "b3"
+		)
+		(pin "b1"
+		)
+		(pin "b18"
+		)
+		(pin "b24"
+		)
+		(pin "b2"
+		)
+		(pin "a1"
+		)
+		(pin "b7"
+		)
+		(pin "b32"
+		)
+		(pin "a21"
+		)
+		(pin "a12"
+		)
+		(pin "b8"
+		)
+		(pin "a20"
+		)
+		(pin "b10"
+		)
+		(pin "b16"
+		)
+		(pin "b5"
+		)
+		(pin "a23"
+		)
+		(pin "a10"
+		)
+		(pin "a32"
+		)
+		(pin "a17"
+		)
+		(pin "a24"
+		)
+		(pin "a19"
+		)
+		(pin "a16"
+		)
+		(pin "a31"
+		)
+		(pin "b15"
+		)
+		(pin "b13"
+		)
+		(pin "a7"
+		)
+		(pin "b20"
+		)
+		(pin "a3"
+		)
+		(pin "b11"
+		)
+		(pin "b21"
+		)
+		(pin "b27"
+		)
+		(pin "b29"
+		)
+		(pin "b25"
+		)
+		(pin "b28"
+		)
+		(pin "b6"
+		)
+		(pin "b23"
+		)
+		(pin "b30"
+		)
+		(pin "a22"
+		)
+		(pin "a8"
+		)
+		(pin "a18"
+		)
+		(pin "b14"
+		)
+		(pin "a30"
+		)
+		(pin "a5"
+		)
+		(pin "a11"
+		)
+		(pin "a4"
+		)
+		(pin "a14"
+		)
+		(pin "a13"
+		)
+		(pin "b31"
+		)
+		(pin "a6"
+		)
+		(pin "b22"
+		)
+		(pin "b26"
+		)
+		(pin "a15"
+		)
+		(pin "a2"
+		)
+		(pin "b19"
+		)
+		(instances
+			(project "cbEval.UIFaceI2C"
+				(path "/7ca35d0c-62a0-45cd-8aba-98caf0370b07"
+					(reference "J13")
+					(unit 1)
+				)
+			)
+		)
 	)
 	(symbol
